Commit message: Fixed bugs after renaming

File: smarc_auvs/models/small_smarc_auv/robots/small_smarc_auv_default.urdf.xacro (robot description, xacro)
@@ -16,5 +16,5 @@
   <xacro:arg name="namespace" default="small_smarc_auv"/>
   <!-- Include the UUV macro file -->
-  <xacro:include filename="$(find small_smarc_auv)/urdf/small_smarc_auv_base.urdf.xacro"/>
+  <xacro:include filename="$(find smarc_auvs)/models/small_smarc_auv/urdf/small_smarc_auv_base.urdf.xacro"/>
   <!-- Create the romulus -->
   <xacro:small_smarc_auv_base namespace="$(arg namespace)" debug="$(arg debug)"/>

File: smarc_auvs/models/small_smarc_auv/urdf/small_smarc_auv_base.urdf.xacro (robot description, xacro)
@@ -26,7 +26,7 @@
   <xacro:property name="cob" value="0 0 0.0196"/>
   <xacro:property name="rho" value="1025.0"/>
-  <xacro:property name="visual_mesh_file" value="file://$(find small_smarc_auv)/mesh/Romulus.dae"/>
-  <xacro:property name="prop_mesh_file" value="file://$(find small_smarc_auv)/mesh/Propeller.dae"/>
-  <xacro:property name="fin_mesh_file" value="file://$(find small_smarc_auv)/mesh/Fin.dae"/>
+  <xacro:property name="visual_mesh_file" value="file://$(find smarc_auvs)/models/small_smarc_auv/mesh/Romulus.dae"/>
+  <xacro:property name="prop_mesh_file" value="file://$(find smarc_auvs)/models/small_smarc_auv/mesh/Propeller.dae"/>
+  <xacro:property name="fin_mesh_file" value="file://$(find smarc_auvs)/models/small_smarc_auv/mesh/Fin.dae"/>
   <!-- Fin snippet -->
   <xacro:macro name="fin_macro" params="namespace fin_id *origin">
