Commit message: Changed the name of the large smarc auv to lolo

File: smarc_auvs/models/lolo_auv/robots/lolo_auv_default.urdf.xacro (robot description, xacro)
@@ -12,11 +12,11 @@
      limitations under the License.
 -->
-<robot name="large_smarc_auv" xmlns:xacro="http://www.ros.org/wiki/xacro" >
+<robot name="lolo_auv" xmlns:xacro="http://www.ros.org/wiki/xacro" >
   <xacro:arg name="debug" default="0"/>
-  <xacro:arg name="namespace" default="large_smarc_auv"/>
+  <xacro:arg name="namespace" default="lolo_auv"/>
   <!-- Include the UUV macro file -->
-  <xacro:include filename="$(find smarc_auvs)/models/large_smarc_auv/urdf/large_smarc_auv_base.urdf.xacro"/>
+  <xacro:include filename="$(find smarc_auvs)/models/lolo_auv/urdf/lolo_auv_base.urdf.xacro"/>
   <!-- Create the romulus -->
-  <xacro:large_smarc_auv_base namespace="$(arg namespace)" debug="$(arg debug)"/>
+  <xacro:lolo_auv_base namespace="$(arg namespace)" debug="$(arg debug)"/>
   <!-- Joint state publisher plugin -->
   <gazebo>

File: smarc_auvs/models/lolo_auv/urdf/lolo_auv_base.urdf.xacro (robot description, xacro)
@@ -26,8 +26,8 @@
   <xacro:property name="cob" value="0 0 0.0196"/>
   <xacro:property name="rho" value="1025.0"/>
-  <xacro:property name="visual_mesh_file" value="file://$(find smarc_auvs)/models/large_smarc_auv/mesh/lolo.dae"/>
-  <xacro:property name="prop_mesh_file" value="file://$(find smarc_auvs)/models/large_smarc_auv/mesh/propeller.dae"/>
-  <xacro:property name="fin_mesh_file" value="file://$(find smarc_auvs)/models/large_smarc_auv/mesh/fin.dae"/>
-  <xacro:property name="back_fin_mesh_file" value="file://$(find smarc_auvs)/models/large_smarc_auv/mesh/back_fin.dae"/>
+  <xacro:property name="visual_mesh_file" value="file://$(find smarc_auvs)/models/lolo_auv/mesh/lolo.dae"/>
+  <xacro:property name="prop_mesh_file" value="file://$(find smarc_auvs)/models/lolo_auv/mesh/propeller.dae"/>
+  <xacro:property name="fin_mesh_file" value="file://$(find smarc_auvs)/models/lolo_auv/mesh/fin.dae"/>
+  <xacro:property name="back_fin_mesh_file" value="file://$(find smarc_auvs)/models/lolo_auv/mesh/back_fin.dae"/>
   <!-- Fin snippet -->
   <xacro:macro name="fin_macro" params="namespace fin_id *origin">
@@ -106,5 +106,5 @@
     </gazebo>
   </xacro:macro>
-  <xacro:macro name="large_smarc_auv_base" params="namespace debug">
+  <xacro:macro name="lolo_auv_base" params="namespace debug">
     <link name="${namespace}/base_link">
       <visual>
