Commit message: Fixed sensors for the lolo auv

File: smarc_auvs/models/lolo_auv/urdf/lolo_auv_base.urdf.xacro (robot description, xacro)
@@ -371,5 +371,5 @@
         scale="0.5">
         <inertia ixx="0.00001" ixy="0.0" ixz="0.0" iyy="0.00001" iyz="0.0" izz="0.00001" />
-        <origin xyz="-0.375 0 -0.16" rpy="0 0.3 0"/>
+        <origin xyz="-0.375 0 -0.3" rpy="0 0.3 0"/>
     </xacro:regular_camera_plugin_macro>
 	<!-- Mount a camera behind the vehicle for steering -->

Commit message: launch file updated for all auvs. Depth sensor add to lolo urdf

File: smarc_auvs/models/lolo_auv/urdf/lolo_auv_base.urdf.xacro (robot description, xacro)
@@ -205,5 +205,5 @@
         </geometry>
       </visual>
-      <collision> -->
+      <collision>
         <!-- todo: gazebo needs a collision volume or it will ignore the pose of
            the joint that leads to this link (and assume it to be the identity) -->
@@ -224,5 +224,5 @@
         </geometry>
       </visual>
-      <collision> -->
+      <collision>
         <!-- todo: gazebo needs a collision volume or it will ignore the pose of
            the joint that leads to this link (and assume it to be the identity) -->
@@ -314,6 +314,6 @@
       topic="sss_left"
       mass="0.015"
-      update_rate="10"
-      samples="120"
+      update_rate="30"
+      samples="102"
       fov="${pi/3.0}"
       range_min="1.0"
@@ -333,6 +333,6 @@
       topic="sss_right"
       mass="0.015"
-      update_rate="10"
-      samples="100"
+      update_rate="30"
+      samples="102"
       fov="${pi/3.0}"
       range_min="1.0"
@@ -349,8 +349,8 @@
       <origin xyz="0 0 0" rpy="0 0 0"/>
     </xacro:default_rpt>  -->
-    <!-- Pressure
+    <!-- Pressure -->
     <xacro:default_pressure namespace="${namespace}" parent_link="${namespace}/base_link">
       <origin xyz="0 0 0" rpy="0 0 0"/>
-    </xacro:default_pressure>  -->
+    </xacro:default_pressure>
     <!-- IMU  -->
     <xacro:default_imu namespace="${namespace}" parent_link="${namespace}/base_link">
