Commit message: Renamed small smarc auv to example auv

File: smarc_auvs/models/example_auv/robots/example_auv_default.urdf.xacro (robot description, xacro)
@@ -12,11 +12,11 @@
      limitations under the License.
 -->
-<robot name="small_smarc_auv" xmlns:xacro="http://www.ros.org/wiki/xacro" >
+<robot name="example_auv" xmlns:xacro="http://www.ros.org/wiki/xacro" >
   <xacro:arg name="debug" default="0"/>
-  <xacro:arg name="namespace" default="small_smarc_auv"/>
+  <xacro:arg name="namespace" default="example_auv"/>
   <!-- Include the UUV macro file -->
-  <xacro:include filename="$(find smarc_auvs)/models/small_smarc_auv/urdf/small_smarc_auv_base.urdf.xacro"/>
+  <xacro:include filename="$(find smarc_auvs)/models/example_auv/urdf/example_auv_base.urdf.xacro"/>
   <!-- Create the romulus -->
-  <xacro:small_smarc_auv_base namespace="$(arg namespace)" debug="$(arg debug)"/>
+  <xacro:example_auv_base namespace="$(arg namespace)" debug="$(arg debug)"/>
   <!-- Joint state publisher plugin -->
   <gazebo>

File: smarc_auvs/models/example_auv/urdf/example_auv_base.urdf.xacro (robot description, xacro)
@@ -27,7 +27,7 @@
   <xacro:property name="cob" value="0 0 0.0196"/>
   <xacro:property name="rho" value="1025.0"/>
-  <xacro:property name="visual_mesh_file" value="file://$(find smarc_auvs)/models/small_smarc_auv/mesh/Romulus.dae"/>
-  <xacro:property name="prop_mesh_file" value="file://$(find smarc_auvs)/models/small_smarc_auv/mesh/Propeller.dae"/>
-  <xacro:property name="fin_mesh_file" value="file://$(find smarc_auvs)/models/small_smarc_auv/mesh/Fin.dae"/>
+  <xacro:property name="visual_mesh_file" value="file://$(find smarc_auvs)/models/example_auv/mesh/Romulus.dae"/>
+  <xacro:property name="prop_mesh_file" value="file://$(find smarc_auvs)/models/example_auv/mesh/Propeller.dae"/>
+  <xacro:property name="fin_mesh_file" value="file://$(find smarc_auvs)/models/example_auv/mesh/Fin.dae"/>
   <!-- Fin snippet -->
   <xacro:macro name="fin_macro" params="namespace fin_id *origin">
@@ -68,5 +68,5 @@
     </gazebo>
   </xacro:macro>
-  <xacro:macro name="small_smarc_auv_base" params="namespace debug">
+  <xacro:macro name="example_auv_base" params="namespace debug">
     <link name="${namespace}/base_link">
       <visual>

Commit message: Changed smarc_auvs refs to smarc_private_auvs

File: smarc_auvs/models/example_auv/robots/example_auv_default.urdf.xacro (robot description, xacro)
@@ -16,5 +16,5 @@
   <xacro:arg name="namespace" default="example_auv"/>
   <!-- Include the UUV macro file -->
-  <xacro:include filename="$(find smarc_auvs)/models/example_auv/urdf/example_auv_base.urdf.xacro"/>
+  <xacro:include filename="$(find smarc_private_auvs)/models/example_auv/urdf/example_auv_base.urdf.xacro"/>
   <!-- Create the romulus -->
   <xacro:example_auv_base namespace="$(arg namespace)" debug="$(arg debug)"/>

File: smarc_auvs/models/example_auv/urdf/example_auv_base.urdf.xacro (robot description, xacro)
@@ -27,7 +27,7 @@
   <xacro:property name="cob" value="0 0 0.0196"/>
   <xacro:property name="rho" value="1025.0"/>
-  <xacro:property name="visual_mesh_file" value="file://$(find smarc_auvs)/models/example_auv/mesh/Romulus.dae"/>
-  <xacro:property name="prop_mesh_file" value="file://$(find smarc_auvs)/models/example_auv/mesh/Propeller.dae"/>
-  <xacro:property name="fin_mesh_file" value="file://$(find smarc_auvs)/models/example_auv/mesh/Fin.dae"/>
+  <xacro:property name="visual_mesh_file" value="file://$(find smarc_private_auvs)/models/example_auv/mesh/Romulus.dae"/>
+  <xacro:property name="prop_mesh_file" value="file://$(find smarc_private_auvs)/models/example_auv/mesh/Propeller.dae"/>
+  <xacro:property name="fin_mesh_file" value="file://$(find smarc_private_auvs)/models/example_auv/mesh/Fin.dae"/>
   <!-- Fin snippet -->
   <xacro:macro name="fin_macro" params="namespace fin_id *origin">
