Commit message: Added the xacro plugin for the forward looking sonar

File: smarc_sensor_plugins/smarc_sensor_plugins_ros/urdf/sonar_snippets.xacro (robot description, xacro)
@@ -89,3 +89,49 @@
   </gazebo>
   </xacro:macro>
+  <xacro:macro name="forward_looking_sonar"
+    params="namespace suffix parent_link topic mass update_rate
+      samples fov width height *inertia *origin *visual">
+    <!-- Sensor link -->
+    <link name="${namespace}/forward_sonar${suffix}_link">
+      <inertial>
+        <xacro:insert_block name="inertia" />
+        <mass value="${mass}" />
+        <origin xyz="0 0 0" rpy="0 0 0" />
+      </inertial>
+      <xacro:insert_block name="visual" />
+      <xacro:no_collision/>
+    </link>
+    <joint name="${namespace}_forward_sonar${suffix}_joint" type="revolute">
+      <xacro:insert_block name="origin" />
+      <parent link="${parent_link}" />
+      <child link="${namespace}/forward_sonar${suffix}_link" />
+      <limit upper="0" lower="0" effort="0" velocity="0" />
+      <axis xyz="1 0 0"/>
+    </joint>
+    <gazebo reference="${namespace}/forward_sonar${suffix}_link">
+      <sensor name="${namespace}/image_sonar" type="depth">
+        <camera>
+		  <horizontal_fov>${fov}</horizontal_fov>
+          <image>
+		    <width>${width}</width>
+		    <height>${height}</height>
+            <format>R8G8B8</format>
+          </image>
+          <clip>
+            <near>0.1</near>
+            <far>17</far>
+          </clip>
+          <save enabled="true">
+            <path>/tmp/camera</path>
+          </save>
+        </camera>
+	    <plugin filename="libimage_sonar_ros_plugin.so" name="forward_sonar${suffix}_controller">
+		  <topicName>${topic}</topicName>
+          <frameName>forward_sonar${suffix}_link</frameName>
+        </plugin>
+        <always_on>true</always_on>
+	    <update_rate>${update_rate}</update_rate>
+      </sensor>
+    </gazebo>
+  </xacro:macro>
 </robot>

Commit message: Fixed the sonar link of the fls

File: smarc_sensor_plugins/smarc_sensor_plugins_ros/urdf/sonar_snippets.xacro (robot description, xacro)
@@ -128,5 +128,5 @@
 	    <plugin filename="libimage_sonar_ros_plugin.so" name="forward_sonar${suffix}_controller">
 		  <topicName>${topic}</topicName>
-          <frameName>forward_sonar${suffix}_link</frameName>
+          <frameName>forward_sonar${suffix}_optical_frame</frameName>
         </plugin>
         <always_on>true</always_on>
@@ -134,4 +134,10 @@
       </sensor>
     </gazebo>
+	<joint name="${namespace}/forward_sonar${suffix}_joint" type="fixed">
+      <origin xyz="0 0 0" rpy="${-pi/2} 0 ${-pi/2}"/>
+      <parent link="${namespace}/forward_sonar${suffix}_link"/>
+      <child link="${namespace}/forward_sonar${suffix}_optical_frame"/>
+    </joint>
+	<link name="${namespace}/forward_sonar${suffix}_optical_frame"/>
   </xacro:macro>
 </robot>

Commit message: Added MBES macro to the sonar_snippets and renamed the SSS macro

File: smarc_sensor_plugins/smarc_sensor_plugins_ros/urdf/sonar_snippets.xacro (robot description, xacro)
@@ -23,5 +23,5 @@
     </collision>
   </xacro:macro>
-  <xacro:macro name="multibeam_intensity_sonar"
+  <xacro:macro name="side_scan_sonar"
     params="namespace suffix parent_link topic mass update_rate
       samples fov range_min range_max range_stddev mesh
@@ -135,3 +135,69 @@
     </gazebo>
   </xacro:macro>
+  <xacro:macro name="multibeam_intensity_sonar"
+    params="namespace suffix parent_link topic mass update_rate
+      samples fov range_min range_max range_stddev mesh
+      *inertia *origin *visual">
+    <!-- Sensor link -->
+    <link name="${namespace}/mbes_sonar${suffix}_link">
+      <inertial>
+        <xacro:insert_block name="inertia" />
+        <mass value="${mass}" />
+        <origin xyz="0 0 0" rpy="0 0 0" />
+      </inertial>
+      <xacro:insert_block name="visual" />
+      <xacro:no_collision/>
+    </link>
+  <joint name="${namespace}_mbes${suffix}_joint" type="revolute">
+    <xacro:insert_block name="origin" />
+    <parent link="${parent_link}" />
+    <child link="${namespace}/mbes_sonar${suffix}_link" />
+    <limit upper="0" lower="0" effort="0" velocity="0" />
+    <axis xyz="1 0 0"/>
+  </joint>
+  <gazebo reference="${namespace}/mbes_sonar${suffix}_link">
+    <sensor type="underwater_sonar" name="mbes_sonar${suffix}">
+      <pose>0 0 0 0 0 0</pose>
+      <visualize>false</visualize>
+      <retro>true</retro>
+      <update_rate>${update_rate}</update_rate>
+      <ray>
+        <scan>
+          <horizontal>
+            <samples>${samples}</samples>
+            <resolution>1</resolution>
+            <min_angle>-${0.5*fov}</min_angle>
+            <max_angle>${0.5*fov}</max_angle>
+          </horizontal>
+		  <vertical>
+		    <resolution>0.5</resolution>
+		    <samples>2</samples>
+			<min_angle>-${0.5*fov/samples}</min_angle>
+            <max_angle>${0.5*fov/samples}</max_angle>
+		  </vertical>
+        </scan>
+        <range>
+          <min>${range_min}</min>
+          <max>${range_max}</max>
+          <resolution>0.01</resolution>
+        </range>
+        <noise>
+          <type>gaussian</type>
+          <mean>0.0</mean>
+          <stddev>${range_stddev}</stddev>
+        </noise>
+      </ray>
+      <plugin name="sonar${suffix}_controller" filename="libunderwater_sonar_ros_plugin.so">
+        <topicName>${topic}</topicName>
+        <frameName>mbes_sonar${suffix}_link</frameName>
+      </plugin>
+      <!-- TODO: Separate switchable sonar version in another macro -->
+	  <!-- <plugin name="switchable_sonar{suffix}_ros_interface" filename="libuuv_gazebo_ros_switchable_gpu_ray_sensor.so">
+          <namespace>${namespace}</namespace>
+          <input_topic>${topic}</input_topic>
+	  </plugin>
+	  -->
+    </sensor>
+  </gazebo>
+  </xacro:macro>
 </robot>

Commit message: Renamed of components of MBES plugin

File: smarc_sensor_plugins/smarc_sensor_plugins_ros/urdf/sonar_snippets.xacro (robot description, xacro)
@@ -36,5 +36,5 @@
       *inertia *origin *visual">
     <!-- Sensor link -->
-    <link name="${namespace}/sonar${suffix}_link">
+    <link name="${namespace}/mbes_sonar${suffix}_link">
       <inertial>
         <xacro:insert_block name="inertia" />
@@ -45,12 +45,12 @@
       <xacro:no_collision/>
     </link>
-  <joint name="${namespace}_sonar${suffix}_joint" type="revolute">
+  <joint name="${namespace}_mbes${suffix}_joint" type="revolute">
     <xacro:insert_block name="origin" />
     <parent link="${parent_link}" />
-    <child link="${namespace}/sonar${suffix}_link" />
+    <child link="${namespace}/mbes_sonar${suffix}_link" />
     <limit upper="0" lower="0" effort="0" velocity="0" />
     <axis xyz="1 0 0"/>
   </joint>
-  <gazebo reference="${namespace}/sonar${suffix}_link">
+  <gazebo reference="${namespace}/mbes_sonar${suffix}_link">
     <sensor type="underwater_sonar" name="sonar${suffix}">
       <pose>0 0 0 0 0 0</pose>
@@ -86,5 +86,5 @@
       <plugin name="sonar${suffix}_controller" filename="libunderwater_sonar_ros_plugin.so">
         <topicName>${topic}</topicName>
-        <frameName>sonar${suffix}_link</frameName>
+        <frameName>mbes_sonar${suffix}_link</frameName>
       </plugin>
       <!-- TODO: Separate switchable sonar version in another macro -->
